File: anavi-thermometer.kicad_sch (KiCad schematic)
At the start: 20 parts, among them J1 USB_B_Micro, P1 CONN_01X03, SW1 SW_DIP_x01, U1 I2C_SENS_1, U2 I2C_SENS_1, U3 I2C_SENS_1, U4 Conn_01x04

Commit message: rev 0.1
Parts:
- removed J1: USB_B_Micro, Connector_USB:USB_Micro-B_Molex-105017-0001, symbol anavi-thermometer-rescue:USB_B_Micro-Connector
- removed R6: 4,7K, Resistor_SMD:R_0603_1608Metric, symbol anavi-thermometer-rescue:R
- removed S2: DS18B20, TerminalBlock_Phoenix:TerminalBlock_Phoenix_MKDS-1,5-3-5.08_1x03_P5.08mm_Horizontal, symbol Sensor_Temperature:DS18B20
- removed U1, U2, U3: I2C_SENS_1, Connector_PinHeader_2.54mm:PinHeader_1x04_P2.54mm_Vertical, symbol anavi-thermometer-rescue:I2C_SENS_1
- removed U4: Conn_01x04, Connector_PinHeader_2.54mm:PinHeader_1x04_P2.54mm_Vertical, symbol Connector_Generic:Conn_01x04
- added J1: USB_A, GCT_USB1061_Horizontal:USB_A_Plug_GCT_USB1061_Horizontal, symbol Connector:USB_A
- added U4: SSD1306, SSD1306:128x64OLED, symbol OLED display:SSD1306
Connections:
- net +3V3: now also U4.2 (VCC)
- net +5V: now also J1.1 (VBUS)
- net GND: now also J1.4 (GND), U4.1 (GND)
- net at ESP-12.13 (GPIO4), R2.2: now also U4.4 (SDA)
- net at ESP-12.14 (GPIO5), R3.2: now also U4.3 (SCL)
- no-connect marks 13 -> 14
Other:
- note added: "SCL"
- note added: "SDA"
- moved on the sheet: C1, C2, D1, ESP-12, P1, R1, R2, R3, R4, R5, S1, SW1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
